Commit message: urdf-file commit

File: src/uarm_description/urdf/uarm2.urdf.xacro (robot description, xacro)
@@ -46,6 +46,16 @@
     <origin xyz="0.15 0 0" rpy="0 0 ${M_PI/2}"/>
       <parent link="${prefix}link_1"/>
+      <child link="${prefix}virtual_link_x"/>
+      <axis xyz="0 0 1"/>
+      <limit effort="200" velocity="1.9634" lower="-${M_PI}" upper="${M_PI}"/>
+    </joint>
+    <link name="${prefix}virtual_link_x">
+    </link>
+    <joint name="${prefix}mimic_joint_x" type="revolute">
+    <origin xyz="0 0 0" rpy="0 0 ${-5*M_PI/8}"/>
+      <parent link="${prefix}virtual_link_x"/>
       <child link="${prefix}link_2"/>
-      <axis xyz="0 0 1"/>
+      <mimic joint="${prefix}joint_1" multiplier="-1"/>
+      <axis xyz="0 0 -1"/>
       <limit effort="200" velocity="1.9634" lower="-${M_PI}" upper="${M_PI}"/>
     </joint>
@@ -58,8 +68,8 @@
     </link>
     <joint name="${prefix}mimic_joint_1" type="revolute">
-    <origin xyz="0.16 0 0" rpy="0 0 ${-M_PI/10}"/>
+    <origin xyz="0.16 0 0" rpy="0 0 ${M_PI/2}"/>
       <parent link="${prefix}link_2"/>
       <child link="${prefix}virtual_link_2"/>
-      <mimic joint="${prefix}joint_1" multiplier="-1"/>
+      <mimic joint="${prefix}joint_1" multiplier="0"/>
       <axis xyz="0 0 -1"/>
       <limit effort="200" velocity="1.9634" lower="-${M_PI}" upper="${M_PI}"/>
@@ -68,5 +78,5 @@
     </link>
     <joint name="${prefix}mimic_joint_2" type="revolute">
-    <origin xyz="0 0 0" rpy="0 0 ${-M_PI/2}"/>
+    <origin xyz="0 0 0" rpy="0 0 ${-7*M_PI/15}"/>
       <parent link="${prefix}virtual_link_2"/>
       <child link="${prefix}link_3"/>
